Commit message: Everything up until LiDAR

File: description/gazebo_control.xacro (robot description, xacro)
@@ -2,5 +2,5 @@
 <robot xmlns:xacro="http://www.ros.org/wiki/xacro">
     <gazebo>
-        <plugin name="diff_drive" filename="libgazebo_ros_diff_drive.so">
+        <plugin name='diff_drive' filename='libgazebo_ros_diff_drive.so'>
          <!-- Wheel Information -->
             <left_joint>left_wheel_joint</left_joint>

File: description/robot.urdf.xacro (robot description, xacro)
@@ -1,6 +1,7 @@
 <?xml version="1.0"?>
-<robot xmlns:xacro="http://www.ros.org/wiki/xacro"  name="robot">
+<robot xmlns:xacro="http://www.ros.org/wiki/xacro" name="robot">
 <xacro:include filename="robot_core.xacro" />
 <xacro:include filename="gazebo_control.xacro"/>
+<!--<xacro:include filename="ros2_control.xacro"/> -->
 <xacro:include filename="lidar.xacro"/>
 <xacro:include filename="camera.xacro"/>

File: description/robot_core.xacro (robot description, xacro)
@@ -19,4 +19,12 @@
     <!-- BASE LINK -->
     <link name="base_link">
+    </link>
+    <!-- BASE FOOTPRINT LINK -->
+    <joint name="base_footprint_joint" type="fixed">
+        <parent link="base_link"/>
+        <child link="base_link"/>
+        <origin xyz="0 0 0" rpy="0 0 0"/>
+    </joint>
+    <link name="base_footprint">
     </link>
     <!-- CHASSIS LINK-->
