Commit message: git push

File: description/robot_core.xacro (robot description, xacro)
@@ -1,3 +1,3 @@
-<?xml version="1.0"?>
+   <?xml version="1.0"?>
 <robot xmlns:xacro="http://www.ros.org/wiki/xacro" >
     <xacro:include filename="inertial_macros.xacro"/>
@@ -17,11 +17,11 @@
         <color rgba="1 0 0 1" />
     </material>
-    <!-- BASE LINK -->
+    <!BASE LINK -->
     <link name="base_link">
     </link>
     <!-- BASE FOOTPRINT LINK -->
-    <joint name="base_footprint_joint" type="fixed">
+   <joint name="base_footprint_joint" type="fixed">
         <parent link="base_link"/>
-        <child link="base_link"/>
+        <child link="base_footprint"/>
         <origin xyz="0 0 0" rpy="0 0 0"/>
     </joint>
@@ -134,3 +134,3 @@
         <mu2 value="0.001"/>
     </gazebo>
-</robot>
+</robot>   -->
